File: schem/schem.sch (KiCad schematic (older format))
At the start: 70 parts, among them U1 ECC83, U2 ECC83, U3 ECC83, U4 ECC83, U5 EL84, U6 EL84

Commit message: Minor modifications
Connections:
- net GND: now also RV1.3
Changed lines of the file:
@@
 Wire Wire Line
 	10350 4900 10350 4750
+$Comp
+L power:GND #PWR?
+U 1 1 5ECAA3E9
+P 3000 2650
+F 0 "#PWR?" H 3000 2400 50  0001 C CNN
+F 1 "GND" H 3005 2477 50  0000 C CNN
+F 2 "" H 3000 2650 50  0001 C CNN
+F 3 "" H 3000 2650 50  0001 C CNN
+	1    3000 2650
+	1    0    0    -1
+$EndComp
+Wire Wire Line
+	3000 2000 3000 2650
 $EndSCHEMATC
